File: board/board.kicad_pcb (KiCad board)
At the start: 2 copper layers, 21 x 13 mm, 1 part

Commit message: initial
Parts:
- removed LOGO1: Logo_Open_Hardware_Small, Symbol:OSHW-Symbol_6.7x6mm_SilkScreen
- added C1: 100n, Capacitor_SMD:C_0603_1608Metric, B.Cu at (83.6, 84.5)
- added C10: 1nF, Capacitor_SMD:C_1825_4564Metric, B.Cu at (97.8, 81.5)
- added C2: 1uF, Capacitor_SMD:C_0603_1608Metric, B.Cu at (93.1, 85.2)
- added C3: 2.2uF, Capacitor_SMD:C_1210_3225Metric, F.Cu at (88.8, 77.9)
- added C4: 10uF, Capacitor_SMD:C_1210_3225Metric, F.Cu at (85.5, 77.9)
- added C5: 1nF, Capacitor_SMD:C_0603_1608Metric, B.Cu at (102.4, 75.0)
- added C6: 47uF, Capacitor_SMD:C_1210_3225Metric, B.Cu at (106.9, 82.8)
- added C7: 47uF, Capacitor_SMD:C_1210_3225Metric, B.Cu at (103.6, 82.8)
- added C8: 220uF, Capacitor_SMD:CP_Elec_10x10.5, F.Cu at (108.0, 94.0)
- added C9: 10n, Capacitor_SMD:C_0805_2012Metric, B.Cu at (85.5, 76.0)
- added D1: 1N4148, Diode_SMD:D_SOD-323, B.Cu at (93.0, 79.8)
- added D2: SBR8U60P5-7, Diode_SMD:D_PowerDI-5, B.Cu at (104.7, 78.1)
- added D3: BAV21, Diode_SMD:D_SOD-323_HandSoldering, B.Cu at (90.1, 76.2)
- added J1: 013_PoE_rectified, on_edge:on_edge_2x05_device, F.Cu at (77.0, 80.6)
- added J2: 003_power, on_edge:on_edge_2x05_host, F.Cu at (114.0, 80.5)
- added L1: 0R, Inductor_SMD:L_1812_4532Metric, F.Cu at (84.1, 84.0)
- added R1: 2.2k, Resistor_SMD:R_0603_1608Metric, B.Cu at (93.1, 82.2)
- added R2: 20k, Resistor_SMD:R_0603_1608Metric, B.Cu at (93.1, 76.5)
- added R3: 41.2R, Resistor_SMD:R_0603_1608Metric, B.Cu at (83.6, 81.5)
- added R4: 24.9k, Resistor_SMD:R_0603_1608Metric, B.Cu at (83.6, 78.5)
- added R5: 49.9k, Resistor_SMD:R_0603_1608Metric, B.Cu at (93.1, 78.0)
- added R6: 105k, Resistor_SMD:R_0603_1608Metric, B.Cu at (93.1, 75.0)
- added R7: 20R, Resistor_SMD:R_0603_1608Metric, B.Cu at (105.5, 75.0)
- added R8: 10K, Resistor_SMD:R_1206_3216Metric, B.Cu at (87.9, 76.5)
- added U1: MP8007, Package_DFN_QFN:QFN-28-1EP_4x5mm_P0.5mm_EP2.65x3.65mm_ThermalVias, B.Cu at (88.0, 83.4)
- added U2: POE70P-50L, local:Transformer_Coilcraft_POE70P, F.Cu at (99.7, 80.5)
Routing:
- net GND: track 0.00 -> 86.2 mm, vias 0 -> 3
- net /flyback/GNDPWR: track 0.00 -> 72.2 mm, vias 0 -> 37
- net /5V: track 0.00 -> 61.5 mm, vias 0 -> 4
- net /3.3V: track 0.00 -> 45.9 mm, vias 0 -> 4
- net /flyback/PoE+: track 0.00 -> 28.2 mm, vias 0 -> 4
- net Net-(C3-Pad1): track 0.00 -> 19.8 mm, vias 0 -> 1
- net Net-(C5-Pad1): track 0.00 -> 16.3 mm, vias 0 -> 2
- net /flyback/PoE-: track 0.00 -> 16.1 mm, vias 0 -> 1
- net Net-(D3-Pad2): track 0.00 -> 12.3 mm, vias 0 -> 3
- net Net-(D1-Pad2): track 0.00 -> 8.50 mm, vias 0 -> 1
- net Net-(R2-Pad1): track 0.00 -> 7.79 mm
- net Net-(R4-Pad2): track 0.00 -> 5.41 mm
- net Net-(C9-Pad2): track 0.00 -> 4.62 mm
- net Net-(R5-Pad1): track 0.00 -> 4.54 mm
- net Net-(C2-Pad1): track 0.00 -> 4.21 mm
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- added copper zone on B.Cu, net /flyback/GNDPWR
- added copper zone on F.Cu, net /flyback/GNDPWR
Other:
- board size 21 x 13 mm -> 37 x 29 mm
- rule pad_to_mask_clearance: 0 -> 0.04
- board text added: "osf.b093.v1.0"
